File: cad/usb415.brd (EAGLE design)
At the start: 45.5 x 15 mm, 40 parts, among them CN1 MICROSD-EJECT, Q1 IRLML6344TRPBF, SW2 SWITCHKMR211, SW3 SWITCHKMR211, U1 STM32F4/64, X1 12MHz, X2 USB-A

Commit message: 2*rgb led, etc
Parts:
- removed LED3: LED, jaw:SMD0603D
- added R12: (no value), jaw:SMD0603
- D1: device jaw:SMD0805D -> jaw:SOD-323
- LED1: device dp_devices:RGBLED -> jaw:SMDLEDRGB
- LED2: value LED -> LED_RGB3; device jaw:SMD0603D -> jaw:SMDLEDRGB
- X2: device adafruit:MOLEX_480371000 -> jaw:MOLEX_480371000
- moved U$2 7.00 mm to (13.0, 23.0)
- moved Q1 3.51 mm to (20.5, 22.5), turned to 270 degrees
- moved LED2 1.50 mm to (13.0, 16.5)
- moved R10 1.50 mm to (17.0, 21.5)
- moved R2 1.50 mm to (17.0, 20.0)
- moved LED1 0.50 mm to (13.0, 13.5)
Connections:
- new net IOLED5: R12.1, U1.26
- new net N$11: LED2.CG, R12.2
- net N$5: now also LED2.CB; no longer LED2.C
- net N$6: now also LED2.CR; no longer LED3.C
- net VCC: now also LED2.AB, LED2.AG, LED2.AR; no longer LED2.A, LED3.A
Routing:
- net IOLED5: track 0.00 -> 16.4 mm, vias 0 -> 2
- net N$14: track 7.16 -> 13.4 mm
- net N$11: track 0.00 -> 2.90 mm
- net N$9: track 3.16 -> 6.02 mm
- net VCC: track 58.1 -> 60.3 mm, vias 7 -> 9
- net IOSPKR: track 15.0 -> 13.6 mm
- net VUSB: track 17.0 -> 17.5 mm
- net GND: vias 17 -> 34
- added copper zone on layer 1, net GND
- added copper zone on layer 16, net GND
- added copper zone on layer 2, net VCC
- removed copper zone on layer 2, net N$10
Other:
- outline, holes or cut-outs redrawn
