File: cad/usb415.sch (EAGLE design)
At the start: 40 parts, among them CN1 MICROSD-EJECT, Q1 IRLML6344TRPBF, SW2 SWITCHKMR211, SW3 SWITCHKMR211, U1 STM32F4/64, X1 12MHz, X2 USB-A

Commit message: 2*rgb led, etc
Parts:
- removed LED3: LED, jaw:LED
- added R12: (no value), jaw:R0603
- D1: device jaw:DIODE-0805 -> jaw:DIODESOD-323
- LED1: device dp_devices:LED_RGB3 -> jaw:LED_RGB3
- LED2: value LED -> LED_RGB3; device jaw:LED -> jaw:LED_RGB3
- X2: device adafruit:USB-A -> jaw:USB-A
Connections:
- new net IOLED5: R12.P$1, U1.PB0
- new net N$11: LED2.CG, R12.P$2
- net N$5: now also LED2.CB; no longer LED2.C
- net N$6: now also LED2.CR; no longer LED3.C
- net VCC: now also LED2.AB, LED2.AG, LED2.AR; no longer LED2.A, LED3.A
Other:
- moved on the sheet: R11, R9
Changed lines of the file:
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@@
 <setting verticaltext="up"/>
 </settings>
-<grid distance="0.1" unitdist="inch" unit="inch" style="lines" multiple="1" display="no" altdistance="0.01" altunitdist="inch" altunit="inch"/>
+<grid distance="0.1" unitdist="inch" unit="inch" style="lines" multiple="1" display="yes" altdistance="0.01" altunitdist="inch" altunit="inch"/>
 <layers>
 <layer number="1" name="Top" color="4" fill="1" visible="no" active="no"/>
@@
 <part name="VCC3" library="jaw" deviceset="PWR-VCC" device=""/>
 <part name="CN1" library="jaw" deviceset="MICROSD" device="-EJECT"/>
-<part name="LED1" library="dp_devices" deviceset="LED_RGB3" device=""/>
+<part name="LED1" library="jaw" deviceset="LED_RGB3" device=""/>
 <part name="SPKR2" library="jaw" deviceset="SPKR" device="-PUI-0440"/>
-<part name="D1" library="jaw" deviceset="DIODE" device="-0805" value="any"/>
+<part name="D1" library="jaw" deviceset="DIODE" device="SOD-323" value="any"/>
 <part name="GND10" library="jaw" deviceset="PWR-GND" device=""/>
 <part name="Q1" library="jaw" deviceset="MOSFET" device="SOT-23" value="IRLML6344TRPBF"/>
@@
 <part name="VCC4" library="jaw" deviceset="PWR-VCC" device=""/>
 <part name="VCC5" library="jaw" deviceset="PWR-VCC" device=""/>
-<part name="LED2" library="jaw" deviceset="LED" device=""/>
 <part name="R9" library="jaw" deviceset="R" device="0603"/>
-<part name="LED3" library="jaw" deviceset="LED" device=""/>
 <part name="R11" library="jaw" deviceset="R" device="0603"/>
 <part name="VCC6" library="jaw" deviceset="PWR-VCC" device=""/>
@@
 <part name="C4" library="jaw" deviceset="C" device="0603" value="2u2"/>
 <part name="VCC8" library="jaw" deviceset="PWR-VCC" device=""/>
-<part name="X2" library="adafruit" deviceset="USB-A" device=""/>
+<part name="X2" library="jaw" deviceset="USB-A" device=""/>
 <part name="U$2" library="adafruit" deviceset="FIDUCIAL" device=""/>
 <part name="U$3" library="adafruit" deviceset="FIDUCIAL" device=""/>
 <part name="LOGO2" library="SparkFun-Aesthetics" deviceset="OSHW-LOGO" device="M"/>
+<part name="LED2" library="jaw" deviceset="LED_RGB3" device=""/>
+<part name="R12" library="jaw" deviceset="R" device="0603"/>
 </parts>
 <sheets>
@@
 <instance part="VCC4" gate="G$1" x="302.26" y="111.76"/>
 <instance part="VCC5" gate="G$1" x="213.36" y="147.32"/>
-<instance part="LED2" gate="G$1" x="284.48" y="86.36" rot="R180"/>
-<instance part="R9" gate="G$1" x="274.32" y="86.36"/>
-<instance part="LED3" gate="G$1" x="284.48" y="76.2" rot="R180"/>
-<instance part="R11" gate="G$1" x="274.32" y="76.2"/>
+<instance part="R9" gate="G$1" x="266.7" y="86.36"/>
+<instance part="R11" gate="G$1" x="266.7" y="83.82"/>
 <instance part="VCC6" gate="G$1" x="269.24" y="175.26"/>
 <instance part="C3" gate="G$1" x="375.92" y="124.46"/>
@@
 <instance part="U$3" gate="G$1" x="408.94" y="25.4"/>
 <instance part="LOGO2" gate="G$1" x="398.78" y="27.94"/>
+<instance part="LED2" gate="G$1" x="284.48" y="83.82"/>
+<instance part="R12" gate="G$1" x="266.7" y="81.28"/>
 </instances>
 <busses>
@@
 <wire x1="302.26" y1="99.06" x2="302.26" y2="101.6" width="0.1524" layer="91"/>
 <junction x="302.26" y="101.6"/>
-<pinref part="LED2" gate="G$1" pin="A"/>
-<wire x1="289.56" y1="86.36" x2="302.26" y2="86.36" width="0.1524" layer="91"/>
+<wire x1="297.18" y1="86.36" x2="302.26" y2="86.36" width="0.1524" layer="91"/>
 <wire x1="302.26" y1="86.36" x2="302.26" y2="99.06" width="0.1524" layer="91"/>
 <junction x="302.26" y="99.06"/>
-<pinref part="LED3" gate="G$1" pin="A"/>
-<wire x1="289.56" y1="76.2" x2="302.26" y2="76.2" width="0.1524" layer="91"/>
-<wire x1="302.26" y1="76.2" x2="302.26" y2="86.36" width="0.1524" layer="91"/>
 <junction x="302.26" y="86.36"/>
+<pinref part="LED2" gate="G$1" pin="AB"/>
+<pinref part="LED2" gate="G$1" pin="AR"/>
+<wire x1="302.26" y1="81.28" x2="302.26" y2="83.82" width="0.1524" layer="91"/>
+<wire x1="302.26" y1="83.82" x2="302.26" y2="86.36" width="0.1524" layer="91"/>
+<wire x1="297.18" y1="83.82" x2="302.26" y2="83.82" width="0.1524" layer="91"/>
+<junction x="302.26" y="83.82"/>
+<pinref part="LED2" gate="G$1" pin="AG"/>
+<wire x1="297.18" y1="81.28" x2="302.26" y2="81.28" width="0.1524" layer="91"/>
 </segment>
 <segment>
@@
 </segment>
 </net>
-<net name="N$5" class="0">
-<segment>
-<pinref part="LED2" gate="G$1" pin="C"/>
-<pinref part="R9" gate="G$1" pin="P$2"/>
-</segment>
-</net>
 <net name="IOLED3" class="0">
 <segment>
 <pinref part="R9" gate="G$1" pin="P$1"/>
-<wire x1="269.24" y1="86.36" x2="264.16" y2="86.36" width="0.1524" layer="91"/>
+<wire x1="261.62" y1="86.36" x2="259.08" y2="86.36" width="0.1524" layer="91"/>
 <label x="254" y="86.36" size="1.27" layer="95" ratio="10"/>
 </segment>
@@
 </segment>
 </net>
-<net name="N$6" class="0">
-<segment>
-<pinref part="LED3" gate="G$1" pin="C"/>
-<pinref part="R11" gate="G$1" pin="P$2"/>
-</segment>
-</net>
 <net name="IOLED4" class="0">
 <segment>
 <pinref part="R11" gate="G$1" pin="P$1"/>
-<wire x1="269.24" y1="76.2" x2="264.16" y2="76.2" width="0.1524" layer="91"/>
-<label x="254" y="76.2" size="1.27" layer="95" ratio="10"/>
+<wire x1="261.62" y1="83.82" x2="259.08" y2="83.82" width="0.1524" layer="91"/>
+<label x="254" y="83.82" size="1.27" layer="95" ratio="10"/>
 </segment>
 <segment>
@@
 </segment>
 </net>
+<net name="IOLED5" class="0">
+<segment>
+<pinref part="U1" gate="G$1" pin="PB0"/>
+<wire x1="160.02" y1="93.98" x2="154.94" y2="93.98" width="0.1524" layer="91"/>
+<label x="147.32" y="93.98" size="1.27" layer="95" ratio="10"/>
+</segment>
+<segment>
+<pinref part="R12" gate="G$1" pin="P$1"/>
+<wire x1="261.62" y1="81.28" x2="259.08" y2="81.28" width="0.1524" layer="91"/>
+<label x="254" y="81.28" size="1.27" layer="95" ratio="10"/>
+</segment>
+</net>
+<net name="N$5" class="0">
+<segment>
+<pinref part="R9" gate="G$1" pin="P$2"/>
+<pinref part="LED2" gate="G$1" pin="CB"/>
+</segment>
+</net>
+<net name="N$6" class="0">
+<segment>
+<pinref part="R11" gate="G$1" pin="P$2"/>
+<pinref part="LED2" gate="G$1" pin="CR"/>
+</segment>
+</net>
+<net name="N$11" class="0">
+<segment>
+<pinref part="LED2" gate="G$1" pin="CG"/>
+<pinref part="R12" gate="G$1" pin="P$2"/>
+</segment>
+</net>

Commit message: R-array
Parts:
- removed R1, R11, R12, R3, R8, R9: (no value), jaw:R0603
- removed R2: 100, jaw:R0603
- added R13, R14: 470, jaw:R-ARRAY40603-ARV
Connections:
- removed net N$11: LED2.CG, R12.P$2
- new net N$10: LED1.CG, R14R.2
- net IOLED0: now also R13B.1; no longer R1.P$1
- net IOLED1: now also R13R.1; no longer R3.P$1
- net IOLED2: now also R13D.1; no longer R8.P$1
- net IOLED3: now also R14A.1; no longer R9.P$1
- net IOLED4: now also R14B.1; no longer R11.P$1
- net IOLED5: now also R14R.1; no longer R12.P$1
- net IOSPKR: now also R14D.1; no longer R2.P$1
- net N$1: now also LED2.CB, R13B.2; no longer LED1.CB, R1.P$2
- net N$2: now also LED2.CR, R13R.2; no longer LED1.CR, R3.P$2
- net N$3: now also LED2.CG, R13D.2; no longer LED1.CG, R8.P$2
- net N$5: now also LED1.CB, R14A.2; no longer LED2.CB, R9.P$2
- net N$6: now also LED1.CR, R14B.2; no longer LED2.CR, R11.P$2
- net N$9: now also R14D.2; no longer R2.P$2
Other:
- note added: "micro SD"
- moved on the sheet: C3, CN1, D1, LED1, LED2, Q1, R10, SPKR2

Commit message: reverse polarity
Connections:
- net GND: now also LED1.CB, LED1.CG, LED1.CR, LED2.CB, LED2.CG, LED2.CR
- net N$1: now also LED1.AG, R14A.2; no longer LED2.CB, R13B.2
- net N$10: now also LED2.AB, R13D.2; no longer LED1.CG, R14R.2
- net N$2: now also LED1.AR, R14B.2; no longer LED2.CR, R13R.2
- net N$3: now also LED1.AB, R14R.2; no longer LED2.CG, R13D.2
- net N$5: now also LED2.AG, R13B.2; no longer LED1.CB, R14A.2
- net N$6: now also LED2.AR, R13R.2; no longer LED1.CR, R14B.2
- net VCC: no longer LED1.AB, LED1.AG, LED1.AR, LED2.AB, LED2.AG, LED2.AR
Other:
- moved on the sheet: LED1, LED2
Changed lines of the file:
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@@
 <part name="VCC3" library="jaw" deviceset="PWR-VCC" device=""/>
 <part name="CN1" library="jaw" deviceset="MICROSD" device="-EJECT"/>
-<part name="LED2" library="jaw" deviceset="LED_RGB3" device=""/>
 <part name="SPKR2" library="jaw" deviceset="SPKR" device="-PUI-0440"/>
 <part name="D1" library="jaw" deviceset="DIODE" device="SOD-323" value="any"/>
@@
 <part name="R10" library="jaw" deviceset="R" device="0603" value="1M"/>
 <part name="VCCA1" library="jaw" deviceset="PWR-VCCA" device=""/>
-<part name="VCC4" library="jaw" deviceset="PWR-VCC" device=""/>
 <part name="VCC5" library="jaw" deviceset="PWR-VCC" device=""/>
 <part name="VCC6" library="jaw" deviceset="PWR-VCC" device=""/>
@@
 <part name="U$3" library="adafruit" deviceset="FIDUCIAL" device=""/>
 <part name="LOGO2" library="SparkFun-Aesthetics" deviceset="OSHW-LOGO" device="M"/>
-<part name="LED1" library="jaw" deviceset="LED_RGB3" device=""/>
 <part name="R13" library="jaw" deviceset="R-ARRAY4" device="0603-ARV" value="470"/>
 <part name="R14" library="jaw" deviceset="R-ARRAY4" device="0603-ARV" value="470"/>
+<part name="LED1" library="jaw" deviceset="LED_RGB3" device=""/>
+<part name="GND2" library="jaw" deviceset="PWR-GND" device=""/>
+<part name="LED2" library="jaw" deviceset="LED_RGB3" device=""/>
 </parts>
 <sheets>
@@
 <instance part="VCC3" gate="G$1" x="233.68" y="175.26"/>
 <instance part="CN1" gate="G$1" x="358.14" y="83.82"/>
-<instance part="LED2" gate="G$1" x="360.68" y="144.78"/>
 <instance part="SPKR2" gate="G$1" x="289.56" y="147.32"/>
 <instance part="D1" gate="G$1" x="279.4" y="147.32" rot="R90"/>
@@
 <instance part="R10" gate="G$1" x="279.4" y="121.92" rot="R270"/>
 <instance part="VCCA1" gate="G$1" x="88.9" y="35.56"/>
-<instance part="VCC4" gate="G$1" x="378.46" y="154.94"/>
 <instance part="VCC5" gate="G$1" x="213.36" y="147.32"/>
 <instance part="VCC6" gate="G$1" x="287.02" y="162.56"/>
@@
 <instance part="U$3" gate="G$1" x="408.94" y="25.4"/>
 <instance part="LOGO2" gate="G$1" x="398.78" y="27.94"/>
-<instance part="LED1" gate="G$1" x="360.68" y="127"/>
 <instance part="R13" gate="A" x="342.9" y="154.94"/>
 <instance part="R13" gate="B" x="342.9" y="147.32"/>
@@
 <instance part="R14" gate="R" x="342.9" y="124.46"/>
 <instance part="R14" gate="D" x="274.32" y="127"/>
+<instance part="LED1" gate="G$1" x="360.68" y="127" rot="R180"/>
+<instance part="GND2" gate="G$1" x="378.46" y="121.92"/>
+<instance part="LED2" gate="G$1" x="360.68" y="144.78" rot="R180"/>
 </instances>
 <busses>
@@
 <label x="378.46" y="68.58" size="1.778" layer="95" ratio="10"/>
 </segment>
+<segment>
+<wire x1="373.38" y1="147.32" x2="378.46" y2="147.32" width="0.1524" layer="91"/>
+<wire x1="373.38" y1="144.78" x2="378.46" y2="144.78" width="0.1524" layer="91"/>
+<wire x1="378.46" y1="144.78" x2="378.46" y2="147.32" width="0.1524" layer="91"/>
+<wire x1="373.38" y1="142.24" x2="378.46" y2="142.24" width="0.1524" layer="91"/>
+<wire x1="378.46" y1="142.24" x2="378.46" y2="144.78" width="0.1524" layer="91"/>
+<junction x="378.46" y="144.78"/>
+<wire x1="373.38" y1="129.54" x2="378.46" y2="129.54" width="0.1524" layer="91"/>
+<wire x1="378.46" y1="129.54" x2="378.46" y2="142.24" width="0.1524" layer="91"/>
+<junction x="378.46" y="142.24"/>
+<junction x="378.46" y="129.54"/>
+<wire x1="378.46" y1="124.46" x2="378.46" y2="127" width="0.1524" layer="91"/>
+<wire x1="378.46" y1="127" x2="378.46" y2="129.54" width="0.1524" layer="91"/>
+<wire x1="373.38" y1="127" x2="378.46" y2="127" width="0.1524" layer="91"/>
+<junction x="378.46" y="127"/>
+<wire x1="373.38" y1="124.46" x2="378.46" y2="124.46" width="0.1524" layer="91"/>
+<pinref part="LED1" gate="G$1" pin="CB"/>
+<pinref part="LED1" gate="G$1" pin="CR"/>
+<pinref part="LED1" gate="G$1" pin="CG"/>
+<pinref part="GND2" gate="G$1" pin="GND"/>
+<junction x="378.46" y="124.46"/>
+<pinref part="LED2" gate="G$1" pin="CB"/>
+<pinref part="LED2" gate="G$1" pin="CR"/>
+<pinref part="LED2" gate="G$1" pin="CG"/>
+</segment>
 </net>
 <net name="VCC" class="0">
@@
 </segment>
 <segment>
-<pinref part="LED2" gate="G$1" pin="AB"/>
-<pinref part="VCC4" gate="G$1" pin="VCC"/>
-<wire x1="373.38" y1="147.32" x2="378.46" y2="147.32" width="0.1524" layer="91"/>
-<wire x1="378.46" y1="147.32" x2="378.46" y2="152.4" width="0.1524" layer="91"/>
-<pinref part="LED2" gate="G$1" pin="AR"/>
-<wire x1="373.38" y1="144.78" x2="378.46" y2="144.78" width="0.1524" layer="91"/>
-<wire x1="378.46" y1="144.78" x2="378.46" y2="147.32" width="0.1524" layer="91"/>
-<junction x="378.46" y="147.32"/>
-<pinref part="LED2" gate="G$1" pin="AG"/>
-<wire x1="373.38" y1="142.24" x2="378.46" y2="142.24" width="0.1524" layer="91"/>
-<wire x1="378.46" y1="142.24" x2="378.46" y2="144.78" width="0.1524" layer="91"/>
-<junction x="378.46" y="144.78"/>
-<wire x1="373.38" y1="129.54" x2="378.46" y2="129.54" width="0.1524" layer="91"/>
-<wire x1="378.46" y1="129.54" x2="378.46" y2="142.24" width="0.1524" layer="91"/>
-<junction x="378.46" y="142.24"/>
-<junction x="378.46" y="129.54"/>
-<pinref part="LED1" gate="G$1" pin="AB"/>
-<pinref part="LED1" gate="G$1" pin="AR"/>
-<wire x1="378.46" y1="124.46" x2="378.46" y2="127" width="0.1524" layer="91"/>
-<wire x1="378.46" y1="127" x2="378.46" y2="129.54" width="0.1524" layer="91"/>
-<wire x1="373.38" y1="127" x2="378.46" y2="127" width="0.1524" layer="91"/>
-<junction x="378.46" y="127"/>
-<pinref part="LED1" gate="G$1" pin="AG"/>
-<wire x1="373.38" y1="124.46" x2="378.46" y2="124.46" width="0.1524" layer="91"/>
-</segment>
-<segment>
 <pinref part="CN1" gate="G$1" pin="VCC"/>
 <wire x1="350.52" y1="76.2" x2="345.44" y2="76.2" width="0.1524" layer="91"/>
@@
 <net name="I2CCL" class="0">
 <segment>
-<wire x1="160.02" y1="78.74" x2="139.7" y2="78.74" width="0.1524" layer="91"/>
-<label x="129.54" y="78.74" size="1.27" layer="95"/>
-<wire x1="139.7" y1="78.74" x2="134.62" y2="78.74" width="0.1524" layer="91"/>
+<wire x1="160.02" y1="78.74" x2="154.94" y2="78.74" width="0.1524" layer="91"/>
+<label x="147.32" y="78.74" size="1.27" layer="95"/>
 <pinref part="U1" gate="G$1" pin="PB6"/>
 </segment>
@@
 <net name="I2CDA" class="0">
 <segment>
-<wire x1="160.02" y1="76.2" x2="144.78" y2="76.2" width="0.1524" layer="91"/>
-<label x="129.54" y="76.2" size="1.27" layer="95"/>
-<wire x1="144.78" y1="76.2" x2="134.62" y2="76.2" width="0.1524" layer="91"/>
+<wire x1="160.02" y1="76.2" x2="154.94" y2="76.2" width="0.1524" layer="91"/>
+<label x="147.32" y="76.2" size="1.27" layer="95"/>
 <pinref part="U1" gate="G$1" pin="PB7"/>
 </segment>
@@
 <net name="N$1" class="0">
 <segment>
-<pinref part="LED2" gate="G$1" pin="CB"/>
+<pinref part="R14" gate="A" pin="2"/>
+<pinref part="LED1" gate="G$1" pin="AG"/>
+</segment>
+</net>
+<net name="N$2" class="0">
+<segment>
+<pinref part="R14" gate="B" pin="2"/>
+<pinref part="LED1" gate="G$1" pin="AR"/>
+</segment>
+</net>
+<net name="N$3" class="0">
+<segment>
+<pinref part="R14" gate="R" pin="2"/>
+<pinref part="LED1" gate="G$1" pin="AB"/>
+</segment>
+</net>
+<net name="N$5" class="0">
+<segment>
 <pinref part="R13" gate="B" pin="2"/>
-</segment>
-</net>
-<net name="N$2" class="0">
-<segment>
-<pinref part="LED2" gate="G$1" pin="CR"/>
+<pinref part="LED2" gate="G$1" pin="AG"/>
+</segment>
+</net>
+<net name="N$6" class="0">
+<segment>
 <pinref part="R13" gate="R" pin="2"/>
-</segment>
-</net>
-<net name="N$3" class="0">
-<segment>
-<pinref part="LED2" gate="G$1" pin="CG"/>
+<pinref part="LED2" gate="G$1" pin="AR"/>
+</segment>
+</net>
+<net name="N$10" class="0">
+<segment>
 <pinref part="R13" gate="D" pin="2"/>
-</segment>
-</net>
-<net name="N$5" class="0">
-<segment>
-<pinref part="LED1" gate="G$1" pin="CB"/>
-<pinref part="R14" gate="A" pin="2"/>
-</segment>
-</net>
-<net name="N$6" class="0">
-<segment>
-<pinref part="LED1" gate="G$1" pin="CR"/>
-<pinref part="R14" gate="B" pin="2"/>
-</segment>
-</net>
-<net name="N$10" class="0">
-<segment>
-<pinref part="LED1" gate="G$1" pin="CG"/>
-<pinref part="R14" gate="R" pin="2"/>
-</segment>
-</net>
+<pinref part="LED2" gate="G$1" pin="AB"/>
+</segment>
+</net>
