File: cad/usb415.sch (EAGLE design)
At the start: 35 parts, among them CN1 MICROSD-EJECT, Q1 IRLML6344TRPBF, SW2 SWITCHKMR211, SW3 SWITCHKMR211, U1 STM32F4/64, X1 12MHz, X2 USB-A

Commit message: eeprom
Parts:
- added U2: EEPROM-I2C-8-DFN8, jaw:EEPROM-I2C-8-DFN8
- R13, R14: value 470 -> 100
Connections:
- net GND: now also U2.A0, U2.A1, U2.A2, U2.GND, U2.WP
- net I2CCL: now also U2.SCL
- net I2CDA: now also U2.SDA
- net VCC: now also U2.VCC
Other:
- note added: "eeprom or ATSHA204"
- note added: "extra resistor, extra fun!"
- moved on the sheet: D1, Q1, R10, R13A, R14D, SPKR2
Changed lines of the file:
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@@
 <part name="U$3" library="adafruit" deviceset="FIDUCIAL" device=""/>
 <part name="LOGO2" library="SparkFun-Aesthetics" deviceset="OSHW-LOGO" device="M"/>
-<part name="R13" library="jaw" deviceset="R-ARRAY4" device="0603-ARV" value="470"/>
-<part name="R14" library="jaw" deviceset="R-ARRAY4" device="0603-ARV" value="470"/>
+<part name="R13" library="jaw" deviceset="R-ARRAY4" device="0603-ARV" value="100"/>
+<part name="R14" library="jaw" deviceset="R-ARRAY4" device="0603-ARV" value="100"/>
 <part name="LED1" library="jaw" deviceset="LED_RGB3" device=""/>
 <part name="GND2" library="jaw" deviceset="PWR-GND" device=""/>
 <part name="LED2" library="jaw" deviceset="LED_RGB3" device=""/>
+<part name="U2" library="jaw" deviceset="EEPROM-I2C-8" device="-DFN8" value="EEPROM-I2C-8-DFN8"/>
+<part name="GND4" library="jaw" deviceset="PWR-GND" device=""/>
+<part name="VCC4" library="jaw" deviceset="PWR-VCC" device=""/>
 </parts>
 <sheets>
 <sheet>
 <plain>
-<wire x1="7.62" y1="45.72" x2="274.32" y2="45.72" width="0.635" layer="97"/>
+<wire x1="7.62" y1="45.72" x2="248.92" y2="45.72" width="0.635" layer="97"/>
 <wire x1="10.16" y1="134.62" x2="86.36" y2="134.62" width="0.635" layer="97"/>
 <wire x1="86.36" y1="134.62" x2="86.36" y2="81.28" width="0.635" layer="97"/>
@@
 <wire x1="312.42" y1="111.76" x2="408.94" y2="111.76" width="0.635" layer="97"/>
 <text x="350.52" y="106.68" size="2.54" layer="97" ratio="10">micro SD</text>
+<wire x1="251.46" y1="111.76" x2="307.34" y2="111.76" width="0.635" layer="97"/>
+<text x="264.16" y="106.68" size="1.778" layer="97" ratio="10">eeprom or ATSHA204</text>
+<text x="350.52" y="157.48" size="1.778" layer="97" ratio="10">extra resistor,
+extra fun!</text>
 </plain>
 <instances>
@@
 <instance part="VCC3" gate="G$1" x="233.68" y="175.26"/>
 <instance part="CN1" gate="G$1" x="358.14" y="83.82"/>
-<instance part="SPKR2" gate="G$1" x="289.56" y="147.32"/>
-<instance part="D1" gate="G$1" x="279.4" y="147.32" rot="R90"/>
-<instance part="GND10" gate="G$1" x="287.02" y="114.3"/>
-<instance part="Q1" gate="G$1" x="287.02" y="129.54"/>
-<instance part="R10" gate="G$1" x="279.4" y="121.92" rot="R270"/>
+<instance part="SPKR2" gate="G$1" x="289.56" y="157.48"/>
+<instance part="D1" gate="G$1" x="279.4" y="157.48" rot="R90"/>
+<instance part="GND10" gate="G$1" x="287.02" y="124.46"/>
+<instance part="Q1" gate="G$1" x="287.02" y="139.7"/>
+<instance part="R10" gate="G$1" x="279.4" y="132.08" rot="R270"/>
 <instance part="VCCA1" gate="G$1" x="88.9" y="35.56"/>
 <instance part="VCC5" gate="G$1" x="213.36" y="147.32"/>
-<instance part="VCC6" gate="G$1" x="287.02" y="162.56"/>
+<instance part="VCC6" gate="G$1" x="287.02" y="172.72"/>
 <instance part="C3" gate="G$1" x="375.92" y="86.36"/>
 <instance part="GND1" gate="G$1" x="375.92" y="81.28"/>
@@
 <instance part="U$3" gate="G$1" x="408.94" y="25.4"/>
 <instance part="LOGO2" gate="G$1" x="398.78" y="27.94"/>
-<instance part="R13" gate="A" x="342.9" y="154.94"/>
+<instance part="R13" gate="A" x="342.9" y="160.02"/>
 <instance part="R13" gate="B" x="342.9" y="147.32"/>
 <instance part="R13" gate="R" x="342.9" y="144.78"/>
@@
 <instance part="R14" gate="B" x="342.9" y="127"/>
 <instance part="R14" gate="R" x="342.9" y="124.46"/>
-<instance part="R14" gate="D" x="274.32" y="127"/>
+<instance part="R14" gate="D" x="274.32" y="137.16"/>
 <instance part="LED1" gate="G$1" x="360.68" y="127" rot="R180"/>
 <instance part="GND2" gate="G$1" x="378.46" y="121.92"/>
 <instance part="LED2" gate="G$1" x="360.68" y="144.78" rot="R180"/>
+<instance part="U2" gate="G$1" x="276.86" y="81.28"/>
+<instance part="GND4" gate="G$1" x="276.86" y="63.5"/>
+<instance part="VCC4" gate="G$1" x="276.86" y="99.06"/>
 </instances>
 <busses>
@@
 <pinref part="Q1" gate="G$1" pin="S"/>
 <pinref part="GND10" gate="G$1" pin="GND"/>
-<wire x1="287.02" y1="124.46" x2="287.02" y2="116.84" width="0.1524" layer="91"/>
+<wire x1="287.02" y1="134.62" x2="287.02" y2="127" width="0.1524" layer="91"/>
 <pinref part="R10" gate="G$1" pin="P$2"/>
-<wire x1="279.4" y1="116.84" x2="287.02" y2="116.84" width="0.1524" layer="91"/>
-<junction x="287.02" y="116.84"/>
+<wire x1="279.4" y1="127" x2="287.02" y2="127" width="0.1524" layer="91"/>
+<junction x="287.02" y="127"/>
 </segment>
 <segment>
@@
 <pinref part="LED2" gate="G$1" pin="CG"/>
 </segment>
+<segment>
+<pinref part="U2" gate="G$1" pin="GND"/>
+<pinref part="GND4" gate="G$1" pin="GND"/>
+</segment>
+<segment>
+<pinref part="U2" gate="G$1" pin="A0"/>
+<wire x1="289.56" y1="83.82" x2="294.64" y2="83.82" width="0.1524" layer="91"/>
+<label x="294.64" y="83.82" size="1.778" layer="95" ratio="10"/>
+</segment>
+<segment>
+<pinref part="U2" gate="G$1" pin="A1"/>
+<wire x1="289.56" y1="81.28" x2="294.64" y2="81.28" width="0.1524" layer="91"/>
+<label x="294.64" y="81.28" size="1.778" layer="95" ratio="10"/>
+</segment>
+<segment>
+<pinref part="U2" gate="G$1" pin="A2"/>
+<wire x1="289.56" y1="78.74" x2="294.64" y2="78.74" width="0.1524" layer="91"/>
+<label x="294.64" y="78.74" size="1.778" layer="95" ratio="10"/>
+</segment>
+<segment>
+<pinref part="U2" gate="G$1" pin="WP"/>
+<wire x1="264.16" y1="83.82" x2="259.08" y2="83.82" width="0.1524" layer="91"/>
+<label x="254" y="83.82" size="1.778" layer="95" ratio="10"/>
+</segment>
 </net>
 <net name="VCC" class="0">
@@
 <segment>
 <pinref part="SPKR2" gate="G$1" pin="P1"/>
-<wire x1="287.02" y1="160.02" x2="287.02" y2="157.48" width="0.1524" layer="91"/>
+<wire x1="287.02" y1="170.18" x2="287.02" y2="167.64" width="0.1524" layer="91"/>
 <pinref part="D1" gate="G$1" pin="C"/>
-<wire x1="279.4" y1="149.86" x2="279.4" y2="157.48" width="0.1524" layer="91"/>
-<wire x1="279.4" y1="157.48" x2="287.02" y2="157.48" width="0.1524" layer="91"/>
-<junction x="287.02" y="157.48"/>
+<wire x1="279.4" y1="160.02" x2="279.4" y2="167.64" width="0.1524" layer="91"/>
+<wire x1="279.4" y1="167.64" x2="287.02" y2="167.64" width="0.1524" layer="91"/>
+<junction x="287.02" y="167.64"/>
 <pinref part="VCC6" gate="G$1" pin="VCC"/>
 </segment>
@@
 <pinref part="U1" gate="G$1" pin="VBAT"/>
 <pinref part="VCC8" gate="G$1" pin="VCC"/>
+</segment>
+<segment>
+<pinref part="U2" gate="G$1" pin="VCC"/>
+<pinref part="VCC4" gate="G$1" pin="VCC"/>
 </segment>
 </net>
@@
 <pinref part="U1" gate="G$1" pin="PB6"/>
 </segment>
+<segment>
+<pinref part="U2" gate="G$1" pin="SCL"/>
+<wire x1="264.16" y1="78.74" x2="259.08" y2="78.74" width="0.1524" layer="91"/>
+<label x="254" y="78.74" size="1.778" layer="95" ratio="10"/>
+</segment>
 </net>
 <net name="I2CDA" class="0">
@@
 <pinref part="U1" gate="G$1" pin="PB7"/>
 </segment>
+<segment>
+<pinref part="U2" gate="G$1" pin="SDA"/>
+<wire x1="264.16" y1="81.28" x2="259.08" y2="81.28" width="0.1524" layer="91"/>
+<label x="254" y="81.28" size="1.778" layer="95" ratio="10"/>
+</segment>
 </net>
 <net name="N$14" class="0">
@@
 <pinref part="Q1" gate="G$1" pin="D"/>
 <pinref part="SPKR2" gate="G$1" pin="P2"/>
-<wire x1="287.02" y1="134.62" x2="287.02" y2="137.16" width="0.1524" layer="91"/>
-<wire x1="287.02" y1="137.16" x2="279.4" y2="137.16" width="0.1524" layer="91"/>
-<junction x="287.02" y="137.16"/>
+<wire x1="287.02" y1="144.78" x2="287.02" y2="147.32" width="0.1524" layer="91"/>
+<wire x1="287.02" y1="147.32" x2="279.4" y2="147.32" width="0.1524" layer="91"/>
+<junction x="287.02" y="147.32"/>
 <pinref part="D1" gate="G$1" pin="A"/>
-<wire x1="279.4" y1="144.78" x2="279.4" y2="137.16" width="0.1524" layer="91"/>
+<wire x1="279.4" y1="154.94" x2="279.4" y2="147.32" width="0.1524" layer="91"/>
 </segment>
 </net>
@@
 <pinref part="Q1" gate="G$1" pin="G"/>
 <pinref part="R10" gate="G$1" pin="P$1"/>
-<wire x1="279.4" y1="127" x2="281.94" y2="127" width="0.1524" layer="91"/>
+<wire x1="279.4" y1="137.16" x2="281.94" y2="137.16" width="0.1524" layer="91"/>
 <pinref part="R14" gate="D" pin="2"/>
-<junction x="279.4" y="127"/>
+<junction x="279.4" y="137.16"/>
 </segment>
 </net>
@@
 <net name="IOSPKR" class="0">
 <segment>
-<wire x1="266.7" y1="127" x2="269.24" y2="127" width="0.1524" layer="91"/>
-<label x="259.08" y="127" size="1.27" layer="95"/>
+<wire x1="266.7" y1="137.16" x2="269.24" y2="137.16" width="0.1524" layer="91"/>
+<label x="259.08" y="137.16" size="1.27" layer="95"/>
 <pinref part="R14" gate="D" pin="1"/>
 </segment>

Commit message: tweak
Parts:
- removed LOGO2: OSHW-LOGOM, SparkFun-Aesthetics:OSHW-LOGOM
- R13, R14: value 100 -> 470
- U2: value EEPROM-I2C-8-DFN8 -> EEPROM-I2C-8-DFN8W; device jaw:EEPROM-I2C-8-DFN8 -> jaw:EEPROM-I2C-8-DFN8W
Other:
- moved on the sheet: U2
Changed lines of the file:
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@@
 <setting verticaltext="up"/>
 </settings>
-<grid distance="0.1" unitdist="inch" unit="inch" style="lines" multiple="1" display="yes" altdistance="0.01" altunitdist="inch" altunit="inch"/>
+<grid distance="0.1" unitdist="inch" unit="inch" style="lines" multiple="1" display="no" altdistance="0.01" altunitdist="inch" altunit="inch"/>
 <layers>
-<layer number="1" name="Top" color="4" fill="1" visible="no" active="no"/>
-<layer number="2" name="Route2" color="1" fill="3" visible="no" active="no"/>
-<layer number="3" name="Route3" color="4" fill="3" visible="no" active="no"/>
-<layer number="14" name="Route14" color="1" fill="6" visible="no" active="no"/>
-<layer number="15" name="Route15" color="4" fill="6" visible="no" active="no"/>
-<layer number="16" name="Bottom" color="1" fill="1" visible="no" active="no"/>
-<layer number="17" name="Pads" color="2" fill="1" visible="no" active="no"/>
-<layer number="18" name="Vias" color="2" fill="1" visible="no" active="no"/>
-<layer number="19" name="Unrouted" color="6" fill="1" visible="no" active="no"/>
-<layer number="20" name="Dimension" color="15" fill="1" visible="no" active="no"/>
-<layer number="21" name="tPlace" color="7" fill="1" visible="no" active="no"/>
-<layer number="22" name="bPlace" color="7" fill="1" visible="no" active="no"/>
-<layer number="23" name="tOrigins" color="15" fill="1" visible="no" active="no"/>
-<layer number="24" name="bOrigins" color="15" fill="1" visible="no" active="no"/>
-<layer number="25" name="tNames" color="7" fill="1" visible="no" active="no"/>
-<layer number="26" name="bNames" color="7" fill="1" visible="no" active="no"/>
-<layer number="27" name="tValues" color="7" fill="1" visible="no" active="no"/>
-<layer number="28" name="bValues" color="7" fill="1" visible="no" active="no"/>
+<layer number="1" name="Top" color="4" fill="1" visible="yes" active="no"/>
+<layer number="2" name="Route2" color="5" fill="1" visible="yes" active="no"/>
+<layer number="3" name="Route3" color="4" fill="3" visible="yes" active="no"/>
+<layer number="14" name="Route14" color="1" fill="6" visible="yes" active="no"/>
+<layer number="15" name="Route15" color="6" fill="1" visible="yes" active="no"/>
+<layer number="16" name="Bottom" color="1" fill="1" visible="yes" active="no"/>
+<layer number="17" name="Pads" color="2" fill="1" visible="yes" active="no"/>
+<layer number="18" name="Vias" color="2" fill="1" visible="yes" active="no"/>
+<layer number="19" name="Unrouted" color="6" fill="1" visible="yes" active="no"/>
+<layer number="20" name="Dimension" color="15" fill="1" visible="yes" active="no"/>
+<layer number="21" name="tPlace" color="7" fill="1" visible="yes" active="no"/>
+<layer number="22" name="bPlace" color="7" fill="1" visible="yes" active="no"/>
+<layer number="23" name="tOrigins" color="15" fill="1" visible="yes" active="no"/>
+<layer number="24" name="bOrigins" color="15" fill="1" visible="yes" active="no"/>
+<layer number="25" name="tNames" color="7" fill="1" visible="yes" active="no"/>
+<layer number="26" name="bNames" color="7" fill="1" visible="yes" active="no"/>
+<layer number="27" name="tValues" color="7" fill="1" visible="yes" active="no"/>
+<layer number="28" name="bValues" color="7" fill="1" visible="yes" active="no"/>
 <layer number="29" name="tStop" color="7" fill="3" visible="no" active="no"/>
 <layer number="30" name="bStop" color="7" fill="6" visible="no" active="no"/>
@@
 <layer number="35" name="tGlue" color="7" fill="4" visible="no" active="no"/>
 <layer number="36" name="bGlue" color="7" fill="5" visible="no" active="no"/>
-<layer number="37" name="tTest" color="7" fill="1" visible="no" active="no"/>
-<layer number="38" name="bTest" color="7" fill="1" visible="no" active="no"/>
+<layer number="37" name="tTest" color="7" fill="1" visible="yes" active="no"/>
+<layer number="38" name="bTest" color="7" fill="1" visible="yes" active="no"/>
 <layer number="39" name="tKeepout" color="4" fill="11" visible="no" active="no"/>
 <layer number="40" name="bKeepout" color="1" fill="11" visible="no" active="no"/>
@@
 <layer number="44" name="Drills" color="7" fill="1" visible="no" active="no"/>
 <layer number="45" name="Holes" color="7" fill="1" visible="no" active="no"/>
-<layer number="46" name="Milling" color="3" fill="1" visible="no" active="no"/>
-<layer number="47" name="Measures" color="7" fill="1" visible="no" active="no"/>
-<layer number="48" name="Document" color="7" fill="1" visible="no" active="no"/>
-<layer number="49" name="Reference" color="7" fill="1" visible="no" active="no"/>
-<layer number="50" name="dxf" color="7" fill="1" visible="no" active="no"/>
-<layer number="51" name="tDocu" color="7" fill="1" visible="no" active="no"/>
-<layer number="52" name="bDocu" color="7" fill="1" visible="no" active="no"/>
-<layer number="53" name="tGND_GNDA" color="7" fill="1" visible="no" active="no"/>
-<layer number="54" name="bGND_GNDA" color="7" fill="1" visible="no" active="no"/>
-<layer number="56" name="wert" color="7" fill="1" visible="no" active="no"/>
-<layer number="57" name="tCAD" color="7" fill="1" visible="no" active="no"/>
-<layer number="59" name="tCarbon" color="7" fill="1" visible="no" active="no"/>
-<layer number="60" name="bCarbon" color="7" fill="1" visible="no" active="no"/>
+<layer number="46" name="Milling" color="3" fill="1" visible="yes" active="no"/>
+<layer number="47" name="Measures" color="7" fill="1" visible="yes" active="no"/>
+<layer number="48" name="Document" color="7" fill="1" visible="yes" active="no"/>
+<layer number="49" name="Reference" color="7" fill="1" visible="yes" active="no"/>
+<layer number="50" name="dxf" color="7" fill="1" visible="yes" active="no"/>
+<layer number="51" name="tDocu" color="7" fill="1" visible="yes" active="no"/>
+<layer number="52" name="bDocu" color="7" fill="1" visible="yes" active="no"/>
+<layer number="53" name="tGND_GNDA" color="7" fill="1" visible="yes" active="no"/>
+<layer number="54" name="bGND_GNDA" color="7" fill="1" visible="yes" active="no"/>
+<layer number="56" name="wert" color="7" fill="1" visible="yes" active="no"/>
+<layer number="57" name="tCAD" color="7" fill="1" visible="yes" active="no"/>
+<layer number="59" name="tCarbon" color="7" fill="1" visible="yes" active="no"/>
+<layer number="60" name="bCarbon" color="7" fill="1" visible="yes" active="no"/>
 <layer number="90" name="Modules" color="5" fill="1" visible="yes" active="yes"/>
 <layer number="91" name="Nets" color="2" fill="1" visible="yes" active="yes"/>
@@
 <part name="U$2" library="adafruit" deviceset="FIDUCIAL" device=""/>
 <part name="U$3" library="adafruit" deviceset="FIDUCIAL" device=""/>
-<part name="LOGO2" library="SparkFun-Aesthetics" deviceset="OSHW-LOGO" device="M"/>
-<part name="R13" library="jaw" deviceset="R-ARRAY4" device="0603-ARV" value="100"/>
-<part name="R14" library="jaw" deviceset="R-ARRAY4" device="0603-ARV" value="100"/>
+<part name="R13" library="jaw" deviceset="R-ARRAY4" device="0603-ARV" value="470"/>
+<part name="R14" library="jaw" deviceset="R-ARRAY4" device="0603-ARV" value="470"/>
 <part name="LED1" library="jaw" deviceset="LED_RGB3" device=""/>
 <part name="GND2" library="jaw" deviceset="PWR-GND" device=""/>
 <part name="LED2" library="jaw" deviceset="LED_RGB3" device=""/>
-<part name="U2" library="jaw" deviceset="EEPROM-I2C-8" device="-DFN8" value="EEPROM-I2C-8-DFN8"/>
+<part name="U2" library="jaw" deviceset="EEPROM-I2C-8" device="-DFN8W" value="EEPROM-I2C-8-DFN8W"/>
 <part name="GND4" library="jaw" deviceset="PWR-GND" device=""/>
 <part name="VCC4" library="jaw" deviceset="PWR-VCC" device=""/>
@@
 <instance part="U$2" gate="G$1" x="408.94" y="33.02"/>
 <instance part="U$3" gate="G$1" x="408.94" y="25.4"/>
-<instance part="LOGO2" gate="G$1" x="398.78" y="27.94"/>
 <instance part="R13" gate="A" x="342.9" y="160.02"/>
 <instance part="R13" gate="B" x="342.9" y="147.32"/>
