File: cad/usb415.sch (EAGLE design)
At the start: 35 parts, among them CN1 MICROSD-EJECT, Q1 IRLML6344TRPBF, SW2 SWITCHKMR211, SW3 SWITCHKMR211, U1 STM32F4/64, U2 EEPROM-I2C-8-DFN8W, X1 12MHz, X2 USB-A

Commit message: tweak
Other:
- moved on the sheet: R13B, R13D, R14A, R14R
Changed lines of the file:
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@@
 <part name="Q1" library="jaw" deviceset="MOSFET" device="SOT-23" value="IRLML6344TRPBF"/>
 <part name="R10" library="jaw" deviceset="R" device="0603" value="1M"/>
-<part name="VCCA1" library="jaw" deviceset="PWR-VCCA" device=""/>
-<part name="VCC5" library="jaw" deviceset="PWR-VCC" device=""/>
 <part name="VCC6" library="jaw" deviceset="PWR-VCC" device=""/>
 <part name="C3" library="jaw" deviceset="C" device="0603" value="4u7"/>
@@
 <part name="U1" library="jaw" deviceset="STM32F4/64" device=""/>
 <part name="C4" library="jaw" deviceset="C" device="0603" value="2u2"/>
-<part name="VCC8" library="jaw" deviceset="PWR-VCC" device=""/>
 <part name="X2" library="jaw" deviceset="USB-A" device=""/>
 <part name="U$2" library="adafruit" deviceset="FIDUCIAL" device=""/>
@@
 <instance part="Q1" gate="G$1" x="287.02" y="139.7"/>
 <instance part="R10" gate="G$1" x="279.4" y="132.08" rot="R270"/>
-<instance part="VCCA1" gate="G$1" x="88.9" y="35.56"/>
-<instance part="VCC5" gate="G$1" x="213.36" y="147.32"/>
 <instance part="VCC6" gate="G$1" x="287.02" y="172.72"/>
 <instance part="C3" gate="G$1" x="375.92" y="86.36"/>
@@
 <instance part="U1" gate="G$1" x="177.8" y="99.06"/>
 <instance part="C4" gate="G$1" x="218.44" y="124.46"/>
-<instance part="VCC8" gate="G$1" x="226.06" y="147.32"/>
 <instance part="X2" gate="G$1" x="25.4" y="106.68"/>
 <instance part="U$2" gate="G$1" x="408.94" y="33.02"/>
 <instance part="U$3" gate="G$1" x="408.94" y="25.4"/>
 <instance part="R13" gate="A" x="342.9" y="160.02"/>
-<instance part="R13" gate="B" x="342.9" y="147.32"/>
+<instance part="R13" gate="B" x="342.9" y="149.86"/>
 <instance part="R13" gate="R" x="342.9" y="144.78"/>
-<instance part="R13" gate="D" x="342.9" y="142.24"/>
-<instance part="R14" gate="A" x="342.9" y="129.54"/>
+<instance part="R13" gate="D" x="342.9" y="139.7"/>
+<instance part="R14" gate="A" x="342.9" y="132.08"/>
 <instance part="R14" gate="B" x="342.9" y="127"/>
-<instance part="R14" gate="R" x="342.9" y="124.46"/>
+<instance part="R14" gate="R" x="342.9" y="121.92"/>
 <instance part="R14" gate="D" x="274.32" y="137.16"/>
 <instance part="LED1" gate="G$1" x="360.68" y="127" rot="R180"/>
@@
 </segment>
 <segment>
-<wire x1="195.58" y1="142.24" x2="203.2" y2="142.24" width="0.1524" layer="91"/>
-<pinref part="VCC2" gate="G$1" pin="VCC"/>
-<wire x1="203.2" y1="142.24" x2="203.2" y2="144.78" width="0.1524" layer="91"/>
-<pinref part="U1" gate="G$1" pin="VCC"/>
-</segment>
-<segment>
 <pinref part="C23" gate="G$1" pin="P$1"/>
 <pinref part="VCC3" gate="G$1" pin="VCC"/>
 </segment>
 <segment>
-<pinref part="VCCA1" gate="G$1" pin="VCCA"/>
-<wire x1="88.9" y1="33.02" x2="88.9" y2="30.48" width="0.1524" layer="91"/>
 <pinref part="C2" gate="G$1" pin="P$1"/>
 <wire x1="60.96" y1="30.48" x2="68.58" y2="30.48" width="0.1524" layer="91"/>
@@
 <pinref part="VR1" gate="G$1" pin="VO"/>
 <wire x1="60.96" y1="30.48" x2="58.42" y2="30.48" width="0.1524" layer="91"/>
-<wire x1="88.9" y1="30.48" x2="76.2" y2="30.48" width="0.1524" layer="91"/>
 </segment>
 <segment>
@@
 <wire x1="350.52" y1="76.2" x2="345.44" y2="76.2" width="0.1524" layer="91"/>
 <label x="340.36" y="76.2" size="1.778" layer="95" ratio="10"/>
-</segment>
-<segment>
-<wire x1="195.58" y1="139.7" x2="213.36" y2="139.7" width="0.1524" layer="91"/>
-<wire x1="213.36" y1="139.7" x2="213.36" y2="144.78" width="0.1524" layer="91"/>
-<pinref part="VCC5" gate="G$1" pin="VCC"/>
-<pinref part="U1" gate="G$1" pin="VCCA"/>
 </segment>
 <segment>
@@
 </segment>
 <segment>
-<wire x1="195.58" y1="137.16" x2="226.06" y2="137.16" width="0.1524" layer="91"/>
-<wire x1="226.06" y1="137.16" x2="226.06" y2="144.78" width="0.1524" layer="91"/>
+<wire x1="195.58" y1="137.16" x2="203.2" y2="137.16" width="0.1524" layer="91"/>
 <pinref part="U1" gate="G$1" pin="VBAT"/>
-<pinref part="VCC8" gate="G$1" pin="VCC"/>
+<wire x1="195.58" y1="139.7" x2="203.2" y2="139.7" width="0.1524" layer="91"/>
+<pinref part="U1" gate="G$1" pin="VCCA"/>
+<wire x1="203.2" y1="137.16" x2="203.2" y2="139.7" width="0.1524" layer="91"/>
+<junction x="203.2" y="139.7"/>
+<wire x1="195.58" y1="142.24" x2="203.2" y2="142.24" width="0.1524" layer="91"/>
+<pinref part="VCC2" gate="G$1" pin="VCC"/>
+<wire x1="203.2" y1="142.24" x2="203.2" y2="144.78" width="0.1524" layer="91"/>
+<pinref part="U1" gate="G$1" pin="VCC"/>
+<wire x1="203.2" y1="139.7" x2="203.2" y2="142.24" width="0.1524" layer="91"/>
+<junction x="203.2" y="142.24"/>
 </segment>
 <segment>
@@
 <net name="IOLED0" class="0">
 <segment>
-<wire x1="337.82" y1="147.32" x2="335.28" y2="147.32" width="0.1524" layer="91"/>
-<label x="330.2" y="147.32" size="1.27" layer="95" ratio="10"/>
+<wire x1="337.82" y1="149.86" x2="335.28" y2="149.86" width="0.1524" layer="91"/>
+<label x="330.2" y="149.86" size="1.27" layer="95" ratio="10"/>
 <pinref part="R13" gate="B" pin="1"/>
 </segment>
@@
 <net name="IOLED2" class="0">
 <segment>
-<wire x1="337.82" y1="142.24" x2="335.28" y2="142.24" width="0.1524" layer="91"/>
-<label x="330.2" y="142.24" size="1.27" layer="95" ratio="10"/>
+<wire x1="337.82" y1="139.7" x2="335.28" y2="139.7" width="0.1524" layer="91"/>
+<label x="330.2" y="139.7" size="1.27" layer="95" ratio="10"/>
 <pinref part="R13" gate="D" pin="1"/>
 </segment>
@@
 <net name="IOLED3" class="0">
 <segment>
-<wire x1="337.82" y1="129.54" x2="335.28" y2="129.54" width="0.1524" layer="91"/>
-<label x="330.2" y="129.54" size="1.27" layer="95" ratio="10"/>
+<wire x1="337.82" y1="132.08" x2="335.28" y2="132.08" width="0.1524" layer="91"/>
+<label x="330.2" y="132.08" size="1.27" layer="95" ratio="10"/>
 <pinref part="R14" gate="A" pin="1"/>
 </segment>
@@
 </segment>
 <segment>
-<wire x1="337.82" y1="124.46" x2="335.28" y2="124.46" width="0.1524" layer="91"/>
-<label x="330.2" y="124.46" size="1.27" layer="95" ratio="10"/>
+<wire x1="337.82" y1="121.92" x2="335.28" y2="121.92" width="0.1524" layer="91"/>
+<label x="330.2" y="121.92" size="1.27" layer="95" ratio="10"/>
 <pinref part="R14" gate="R" pin="1"/>
 </segment>
@@
 <pinref part="R14" gate="A" pin="2"/>
 <pinref part="LED1" gate="G$1" pin="AG"/>
+<wire x1="347.98" y1="132.08" x2="347.98" y2="129.54" width="0.1524" layer="91"/>
 </segment>
 </net>
@@
 <pinref part="R14" gate="R" pin="2"/>
 <pinref part="LED1" gate="G$1" pin="AB"/>
+<wire x1="347.98" y1="121.92" x2="347.98" y2="124.46" width="0.1524" layer="91"/>
 </segment>
 </net>
@@
 <pinref part="R13" gate="B" pin="2"/>
 <pinref part="LED2" gate="G$1" pin="AG"/>
+<wire x1="347.98" y1="149.86" x2="347.98" y2="147.32" width="0.1524" layer="91"/>
 </segment>
 </net>
@@
 <pinref part="R13" gate="D" pin="2"/>
 <pinref part="LED2" gate="G$1" pin="AB"/>
-</segment>
-</net>
+<wire x1="347.98" y1="139.7" x2="347.98" y2="142.24" width="0.1524" layer="91"/>
+</segment>
+</net>

Commit message: sd connector
Parts:
- removed C21: .1u, jaw:C0603
- removed C22: 4u7, jaw:C0603
- removed R10: 1M, jaw:R0603
- removed R13, R14: 470, jaw:R-ARRAY40603-ARV
- removed SW3: SWITCHKMR211, jaw:SWITCHKMR211
- added C5, C6: 2u2, jaw:C0603
- added R1, R2: 10k, jaw:R0603
- added R3: 22, jaw:R0603
- added SW1: SWITCHKMR211, jaw:SWITCHKMR211
- C10: value 2u2 -> .1u
- C11: value 10u -> 4u7
- C3: value 4u7 -> 10u
- C4: value 2u2 -> 4u7
- CN1: value MICROSD-EJECT -> MICROSDPLAIN; device jaw:MICROSD-EJECT -> jaw:MICROSDPLAIN
- R4: value 10k -> 22
- R5: value 10k -> 1M
- R6, R7: value 22 -> 470; device jaw:R0603 -> jaw:R-ARRAY40603-ARV
- renumbered C15 to C7, C19 to C8, C20 to C9, C23 to C12, SPKR2 to SPKR1
Connections:
- net BOOT0: now also R1.P$2, SW2.P$2; no longer R4.P$2, SW3.P$2
- net GND: now also C5.P$2, C6.P$2, R1.P$1, R5.P$2, SW1.P$1; no longer C21.P$2, C22.P$2, R10.P$2, R4.P$1, SW2.P$1
- net IOLED0: now also R6B.1; no longer R13B.1
- net IOLED1: now also R6R.1; no longer R13R.1
- net IOLED2: now also R6D.1; no longer R13D.1
- net IOLED3: now also R7A.1; no longer R14A.1
- net IOLED4: now also R7B.1; no longer R14B.1
- net IOLED5: now also R7R.1; no longer R14R.1
- net IOSPKR: now also R7D.1; no longer R14D.1
- net N$1: now also R7A.2; no longer R14A.2
- net N$10: now also R6D.2; no longer R13D.2
- net N$18: now also C5.P$1; no longer C10.P$1
- net N$2: now also R7B.2; no longer R14B.2
- net N$3: now also R7R.2; no longer R14R.2
- net N$4: now also C6.P$1; no longer C4.P$1
- net N$5: now also R6B.2; no longer R13B.2
- net N$6: now also R6R.2; no longer R13R.2
- net N$7: now also R4.P$1; no longer R6.P$1
- net N$8: now also R3.P$1; no longer R7.P$1
- net N$9: now also R5.P$1, R7D.2; no longer R10.P$1, R14D.2
- net NRST: now also R2.P$1, SW1.P$2; no longer R5.P$1, SW2.P$2
- net USBDM: now also R4.P$2; no longer R6.P$2
- net USBDP: now also R3.P$2; no longer R7.P$2
- net VCC: now also C10.P$1, C4.P$1, R2.P$2, SW2.P$1; no longer C21.P$1, C22.P$1, R5.P$2, SW3.P$1
Other:
- moved on the sheet: C10, C11, C3, C4, CN1, R4, R5, SW2

Commit message: add prog/test header
Parts:
- added CN2: HEADER-3X2-PTH1.27, jaw:HEADER-3X2-PTH1.27
Connections:
- new net RX: CN2.P$3, U1.PB11
- new net TX: CN2.P$4, U1.PB10
- net BOOT0: now also CN2.P$5
- net GND: now also CN2.P$2
- net IOSPKR: now also U1.PA3; no longer U1.PB11
- net NRST: now also CN2.P$6
- net VUSB: now also CN2.P$1
Other:
- note added: "programming/testing"
- moved on the sheet: LED2, R6A, R6B, R6D, R6R, R7A, R7R
