File: cad/cryptojawn.sch (EAGLE design)
At the start: 36 parts, among them CN1 MICROSDPLAIN, CN2 HEADER-3X2-PTH1.27, Q1 IRLML6344TRPBF, SW1 SWITCHKMR211, SW2 SWITCHKMR211, U1 STM32F4/64, U2 EEPROM-I2C-8-DFN8W, X1 12MHz, X2 USB-A

Commit message: hardware rev.1
Parts:
- removed D1: any, jaw:DIODESOD-323
- removed LED2: LED_RGB3, jaw:LED_RGB3
- removed X2: USB-A, jaw:USB-A
- added CN10, CN11, CN4, CN5, CN6, CN7, CN8, CN9: HEADER-1X1-SPOT, jaw-conn:HEADER-1X1-SPOT
- added CN3: USB-A-2100, jaw-conn:USB-A-2100
- added R8: 470, jaw:R0603
- added SW3: SWITCH-PTS810, jaw:SWITCH-PTS810
- added U$4: FIDUCIAL, adafruit:FIDUCIAL
- CN2: value HEADER-3X2-PTH1.27 -> DO NOT PLACE; device jaw:HEADER-3X2-PTH1.27 -> jaw-conn:HEADER-3X2-PTH1.27
- LED1: value LED_RGB3 -> LED-RGB-CA-PLCC4; device jaw:LED_RGB3 -> jaw:LED-RGB-CA-PLCC4
- Q1: value IRLML6344TRPBF -> MOSFET-2N; device jaw:MOSFETSOT-23 -> jaw:MOSFET-2N
- R6, R7: device jaw:R-ARRAY40603-ARV -> jaw:R0603
- SW1, SW2: value SWITCHKMR211 -> SWITCH-PTS810; device jaw:SWITCHKMR211 -> jaw:SWITCH-PTS810
Connections:
- removed net N$10: LED2.AB, R6D.2
- removed net N$6: LED2.AR, R6R.2
- removed net N$9: Q1.G, R5.P$1, R7D.2
- new net IOTEST: CN11.P$1, U1.PA4
- net BOOT0: now also CN2.P$4, CN8.P$1; no longer CN2.P$5
- net GND: now also CN2.P$1, CN3.GND, CN5.P$1, Q1G$1.S; no longer CN2.P$2, LED1.CB, LED1.CG, LED1.CR, LED2.CB, LED2.CG, LED2.CR, Q1.S, X2.GND
- net IOLED0: now also R6.P$1; no longer R6B.1
- net IOLED1: now also R7.P$1; no longer R6R.1
- net IOLED2: now also R8.P$1; no longer R6D.1
- net IOLED3: no longer R7A.1
- net IOLED4: no longer R7B.1
- net IOLED5: no longer R7R.1
- net IOSPKR: now also Q1G$1.G, R5.P$1; no longer R7D.1
- net N$1: now also LED1.CB, R7.P$2; no longer LED1.AG, R7A.2
- net N$14: now also Q1G$1.D, Q1G$2.G, Q1G$2.S; no longer D1.A, Q1.D
- net N$2: now also SW3.P$1, U1.PB15; no longer LED1.AR, R7B.2
- net N$3: now also LED1.CR, R8.P$2; no longer LED1.AB, R7R.2
- net N$5: now also LED1.CG, R6.P$2; no longer LED2.AG, R6B.2
- net N$7: now also CN3.D-; no longer X2.D-
- net N$8: now also CN3.D+; no longer X2.D+
- net NRST: now also CN9.P$1
- net RX: now also CN2.P$5, CN7.P$1; no longer CN2.P$3
- net TX: now also CN2.P$3, CN6.P$1; no longer CN2.P$4
- net VCC: now also CN10.P$1, LED1.A, Q1G$2.D, SW3.P$2; no longer D1.C
- net VUSB: now also CN2.P$2, CN3.VBUS, CN4.P$1; no longer CN2.P$1, X2.VBUS
Other:
- note added: "(diode)"
- note added: "eeprom or ATSHA204, ATECC608, etc"
- note removed: "eeprom or ATSHA204"
- note removed: "extra resistor, extra fun!"
- moved on the sheet: CN2

Commit message: misc
Parts:
- CN3: value USB-A-2100 -> USB-A-2100-H; device jaw-conn:USB-A-2100 -> jaw-conn:USB-A-2100-H
- Q1: value MOSFET-2N -> DMN63D8LDW
- U1: device jaw:STM32F4/64 -> jaw-ic:STM32F4/64
Connections:
- new net N$10: U1.PC1
- new net N$11: U1.PC2
- new net N$15: U1.PC3
- new net N$9: U1.PC0
- net N$2: now also U1.PB13; no longer U1.PB15
- net USBDM: now also U1.PB14
- net USBDP: now also U1.PB15
Other:
- note added: "B2=boot1"
- note added: "board detect"
- moved on the sheet: SW3
Changed lines of the file:
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@@
 <part name="VCC7" library="jaw" deviceset="PWR-VCC" device=""/>
 <part name="U$1" library="jaw" deviceset="ROBOTMAN-LOGO" device=""/>
-<part name="U1" library="jaw" deviceset="STM32F4/64" device=""/>
+<part name="U1" library="jaw-ic" deviceset="STM32F4/64" device=""/>
 <part name="C6" library="jaw" deviceset="C" device="0603" value="2u2"/>
-<part name="CN3" library="jaw-conn" deviceset="USB-A" device="-2100"/>
+<part name="CN3" library="jaw-conn" deviceset="USB-A" device="-2100-H" value="USB-A-2100-H"/>
 <part name="U$2" library="adafruit" deviceset="FIDUCIAL" device=""/>
 <part name="U$3" library="adafruit" deviceset="FIDUCIAL" device=""/>
@@
 <part name="LED1" library="jaw" deviceset="LED-RGB-CA" device="-PLCC4"/>
 <part name="VCC8" library="jaw" deviceset="PWR-VCC" device=""/>
-<part name="Q1" library="jaw" deviceset="MOSFET-2N" device=""/>
+<part name="Q1" library="jaw" deviceset="MOSFET-2N" device="" value="DMN63D8LDW"/>
 <part name="CN4" library="jaw-conn" deviceset="HEADER-1X1" device="-SPOT"/>
 <part name="CN5" library="jaw-conn" deviceset="HEADER-1X1" device="-SPOT"/>
@@
 <wire x1="248.92" y1="43.18" x2="248.92" y2="2.54" width="0.635" layer="97"/>
 <text x="261.62" y="157.48" size="1.778" layer="97">(diode)</text>
+<text x="134.62" y="88.9" size="1.27" layer="97">B2=boot1</text>
+<text x="147.32" y="68.58" size="1.27" layer="97">board
+detect</text>
 </plain>
 <instances>
@@
 <instance part="VCC4" gate="G$1" x="276.86" y="99.06"/>
 <instance part="CN2" gate="G$1" x="264.16" y="20.32"/>
-<instance part="SW3" gate="G$1" x="218.44" y="76.2"/>
+<instance part="SW3" gate="G$1" x="218.44" y="81.28"/>
 <instance part="R6" gate="G$1" x="342.9" y="160.02"/>
 <instance part="R7" gate="G$1" x="342.9" y="149.86"/>
 <instance part="R8" gate="G$1" x="342.9" y="139.7"/>
-<instance part="VCC5" gate="G$1" x="226.06" y="78.74"/>
+<instance part="VCC5" gate="G$1" x="228.6" y="83.82"/>
 <instance part="LED1" gate="G$1" x="353.06" y="149.86" rot="R180"/>
 <instance part="VCC8" gate="G$1" x="363.22" y="152.4"/>
@@
 <pinref part="SW3" gate="G$1" pin="P$2"/>
 <pinref part="VCC5" gate="G$1" pin="VCC"/>
+<wire x1="226.06" y1="81.28" x2="228.6" y2="81.28" width="0.1524" layer="91"/>
 </segment>
 <segment>
@@
 <pinref part="U1" gate="G$1" pin="PA11"/>
 </segment>
+<segment>
+<pinref part="U1" gate="G$1" pin="PB14"/>
+<wire x1="195.58" y1="78.74" x2="200.66" y2="78.74" width="0.1524" layer="91"/>
+<label x="200.66" y="78.74" size="1.27" layer="95"/>
+</segment>
 </net>
 <net name="USBDP" class="0">
@@
 <label x="200.66" y="106.68" size="1.27" layer="95"/>
 <pinref part="U1" gate="G$1" pin="PA12"/>
+</segment>
+<segment>
+<pinref part="U1" gate="G$1" pin="PB15"/>
+<wire x1="195.58" y1="76.2" x2="200.66" y2="76.2" width="0.1524" layer="91"/>
+<label x="200.66" y="76.2" size="1.27" layer="95"/>
 </segment>
 </net>
@@
 </segment>
 </net>
-<net name="N$2" class="0">
-<segment>
-<pinref part="U1" gate="G$1" pin="PB15"/>
-<pinref part="SW3" gate="G$1" pin="P$1"/>
-<wire x1="195.58" y1="76.2" x2="213.36" y2="76.2" width="0.1524" layer="91"/>
-</segment>
-</net>
 <net name="N$1" class="0">
 <segment>
@@
 </segment>
 </net>
+<net name="N$2" class="0">
+<segment>
+<pinref part="U1" gate="G$1" pin="PB13"/>
+<pinref part="SW3" gate="G$1" pin="P$1"/>
+<wire x1="195.58" y1="81.28" x2="213.36" y2="81.28" width="0.1524" layer="91"/>
+</segment>
+</net>
+<net name="N$9" class="0">
+<segment>
+<pinref part="U1" gate="G$1" pin="PC0"/>
+<wire x1="160.02" y1="71.12" x2="154.94" y2="71.12" width="0.1524" layer="91"/>
+</segment>
+</net>
+<net name="N$10" class="0">
+<segment>
+<pinref part="U1" gate="G$1" pin="PC1"/>
+<wire x1="160.02" y1="68.58" x2="154.94" y2="68.58" width="0.1524" layer="91"/>
+</segment>
+</net>
+<net name="N$11" class="0">
+<segment>
+<pinref part="U1" gate="G$1" pin="PC2"/>
+<wire x1="160.02" y1="66.04" x2="154.94" y2="66.04" width="0.1524" layer="91"/>
+</segment>
+</net>
+<net name="N$15" class="0">
+<segment>
+<pinref part="U1" gate="G$1" pin="PC3"/>
+<wire x1="160.02" y1="63.5" x2="154.94" y2="63.5" width="0.1524" layer="91"/>
+</segment>
+</net>
